File: minimouse.kicad_sch (KiCad schematic)
At the start: 1 part

Commit message: heyo
Parts:
- removed R13: 100, Resistor_SMD:R_0603_1608Metric, symbol Device:R
Changed lines of the file:
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@@
     (stroke (width 0) (type default))
   )
-  (wire (pts (xy 100.33 107.95) (xy 105.41 107.95))
-    (stroke (width 0) (type default))
-  )
-  (wire (pts (xy 87.63 107.95) (xy 92.71 107.95))
+  (wire (pts (xy 87.63 107.95) (xy 105.41 107.95))
     (stroke (width 0) (type default))
   )
@@
     (stroke (width 0) (type default))
   )
-  (symbol (lib_id "Device:R") (at 96.52 107.95 90) (unit 1)
-    (in_bom yes) (on_board yes) (dnp no) (fields_autoplaced)
-    (property "Reference" "R13" (at 96.52 101.6 90)
-      (effects (font (size 1.27 1.27)))
-    )
-    (property "Value" "100" (at 96.52 104.14 90)
-      (effects (font (size 1.27 1.27)))
-    )
-    (property "Footprint" "Resistor_SMD:R_0603_1608Metric" (at 96.52 109.728 90)
-      (effects (font (size 1.27 1.27)) hide)
-    )
-    (property "Datasheet" "~" (at 96.52 107.95 0)
-      (effects (font (size 1.27 1.27)) hide)
-    )
-    (pin "1")
-    (pin "2")
-    (instances
-      (project "minimouse"
-        (path "/d8fa4cba-2469-4231-847f-065b6b829f44"
-          (reference "R13") (unit 1)
-        )
-      )
-    )
-  )
   (sheet (at 163.83 69.85) (size 34.29 25.4) (fields_autoplaced)

Commit message: tp2
Parts:
- added R13: 100, symbol Device:R
Connections:
- net external_uart/EXT_UART_RX: now also R13.1
- new net mcu/UART1_TX: R13.2
Changed lines of the file:
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@@
     (stroke (width 0) (type default))
   )
-  (wire (pts (xy 87.63 107.95) (xy 105.41 107.95))
+  (wire (pts (xy 100.33 107.95) (xy 105.41 107.95))
+    (stroke (width 0) (type default))
+  )
+  (wire (pts (xy 87.63 107.95) (xy 92.71 107.95))
     (stroke (width 0) (type default))
   )
@@
     (stroke (width 0) (type default))
   )
+  (symbol (lib_id "Device:R") (at 96.52 107.95 90) (unit 1)
+    (in_bom yes) (on_board yes) (dnp no) (fields_autoplaced)
+    (property "Reference" "R13" (at 96.52 101.6 90)
+      (effects (font (size 1.27 1.27)))
+    )
+    (property "Value" "100" (at 96.52 104.14 90)
+      (effects (font (size 1.27 1.27)))
+    )
+    (property "Footprint" "" (at 96.52 109.728 90)
+      (effects (font (size 1.27 1.27)) hide)
+    )
+    (property "Datasheet" "~" (at 96.52 107.95 0)
+      (effects (font (size 1.27 1.27)) hide)
+    )
+    (pin "1")
+    (pin "2")
+    (instances
+      (project "minimouse"
+        (path "/d8fa4cba-2469-4231-847f-065b6b829f44"
+          (reference "R13") (unit 1)
+        )
+      )
+    )
+  )
   (sheet (at 163.83 69.85) (size 34.29 25.4) (fields_autoplaced)

Commit message: test
Parts:
- R13: footprint (none) -> Resistor_SMD:R_0603_1608Metric
Changed lines of the file:
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@@
       (effects (font (size 1.27 1.27)))
     )
-    (property "Footprint" "" (at 96.52 109.728 90)
+    (property "Footprint" "Resistor_SMD:R_0603_1608Metric" (at 96.52 109.728 90)
       (effects (font (size 1.27 1.27)) hide)
     )
