File: mm_mcu.kicad_sch (KiCad schematic)
At the start: 18 parts, among them J1 Conn_ARM_JTAG_SWD_10, U1 STM32F030C8Tx

Commit message: test
Changed lines of the file:
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@@
     )
     (property "Value" "2.2uF" (at 214.63 36.83 0)
-      (effects (font (size 1.27 1.27)) (justify left))
+      (effects (font (size 1.27 1.27)) (justify left) hide)
     )
     (property "Footprint" "Capacitor_SMD:C_0603_1608Metric" (at 214.3252 38.1 0)
@@
     )
     (property "Value" "0.1uF" (at 231.14 36.83 0)
-      (effects (font (size 1.27 1.27)) (justify left))
+      (effects (font (size 1.27 1.27)) (justify left) hide)
     )
     (property "Footprint" "Capacitor_SMD:C_0603_1608Metric" (at 230.8352 38.1 0)
@@
     )
     (property "Value" "100" (at 120.65 76.2 90)
-      (effects (font (size 1.27 1.27)))
+      (effects (font (size 1.27 1.27)) hide)
     )
     (property "Footprint" "Resistor_SMD:R_0603_1608Metric" (at 115.57 79.248 90)
@@
     )
     (property "Value" "100" (at 171.45 53.34 90)
-      (effects (font (size 1.27 1.27)))
+      (effects (font (size 1.27 1.27)) hide)
     )
     (property "Footprint" "Resistor_SMD:R_0603_1608Metric" (at 166.37 56.388 90)
@@
     )
     (property "Value" "100" (at 120.65 73.66 90)
-      (effects (font (size 1.27 1.27)))
+      (effects (font (size 1.27 1.27)) hide)
     )
     (property "Footprint" "Resistor_SMD:R_0603_1608Metric" (at 115.57 76.708 90)
@@
     )
     (property "Value" "100" (at 120.65 88.9 90)
-      (effects (font (size 1.27 1.27)))
+      (effects (font (size 1.27 1.27)) hide)
     )
     (property "Footprint" "Resistor_SMD:R_0603_1608Metric" (at 115.57 91.948 90)
@@
     )
     (property "Value" "100" (at 171.45 45.72 90)
-      (effects (font (size 1.27 1.27)))
+      (effects (font (size 1.27 1.27)) hide)
     )
     (property "Footprint" "Resistor_SMD:R_0603_1608Metric" (at 166.37 48.768 90)
@@
     )
     (property "Value" "100" (at 120.65 96.52 90)
-      (effects (font (size 1.27 1.27)))
+      (effects (font (size 1.27 1.27)) hide)
     )
     (property "Footprint" "Resistor_SMD:R_0603_1608Metric" (at 115.57 99.568 90)
@@
     )
     (property "Value" "100" (at 171.45 48.26 90)
-      (effects (font (size 1.27 1.27)))
+      (effects (font (size 1.27 1.27)) hide)
     )
     (property "Footprint" "Resistor_SMD:R_0603_1608Metric" (at 166.37 51.308 90)
@@
     )
     (property "Value" "0.1uF" (at 248.92 36.83 0)
-      (effects (font (size 1.27 1.27)) (justify left))
+      (effects (font (size 1.27 1.27)) (justify left) hide)
     )
     (property "Footprint" "Capacitor_SMD:C_0603_1608Metric" (at 248.6152 38.1 0)
@@
     )
     (property "Value" "0.1uF" (at 257.81 36.83 0)
-      (effects (font (size 1.27 1.27)) (justify left))
+      (effects (font (size 1.27 1.27)) (justify left) hide)
     )
     (property "Footprint" "Capacitor_SMD:C_0603_1608Metric" (at 257.5052 38.1 0)
@@
     )
     (property "Value" "0.1uF" (at 240.03 36.83 0)
-      (effects (font (size 1.27 1.27)) (justify left))
+      (effects (font (size 1.27 1.27)) (justify left) hide)
     )
     (property "Footprint" "Capacitor_SMD:C_0603_1608Metric" (at 239.7252 38.1 0)
@@
     )
     (property "Value" "100" (at 171.45 50.8 90)
-      (effects (font (size 1.27 1.27)))
+      (effects (font (size 1.27 1.27)) hide)
     )
     (property "Footprint" "Resistor_SMD:R_0603_1608Metric" (at 166.37 53.848 90)
@@
     )
     (property "Value" "2.2uF" (at 222.25 36.83 0)
-      (effects (font (size 1.27 1.27)) (justify left))
+      (effects (font (size 1.27 1.27)) (justify left) hide)
     )
     (property "Footprint" "Capacitor_SMD:C_0603_1608Metric" (at 221.9452 38.1 0)
