File: mm_motor_control.kicad_sch (KiCad schematic)
At the start: 0 parts

Commit message: tp2
Parts:
- added C7: 10n, symbol Device:C
- added C8: 22n, symbol Device:C
- added C9: C, symbol Device:C
- added C_Pol: 20µ, symbol Device:C_Polarized
- added Cs: 2.2µ, symbol Device:C
- added R10, RsnsA: 330m, symbol Device:R
- added R11: 10k, symbol Device:R
- added REN: 18k, symbol Device:R
- added ROFF: 47k, symbol Device:R
- added RRCOFF: 1k, symbol Device:R
- added U4: STSPIN240, Package_DFN_QFN:VQFN-16-1EP_3x3mm_P0.5mm_EP1.8x1.8mm, symbol Driver_Motor:STSPIN240
Connections:
- net EN: now also REN.1
- net OUT_A1: now also U4.3 (OUTA1)
- net OUT_A2: now also U4.5 (OUTA2)
- net OUT_B1: now also U4.10 (OUTB1)
- net OUT_B2: now also U4.8 (OUTB2)
- net PHASE_A: now also U4.1 (PHA)
- net PHASE_B: now also U4.15 (PHB)
- net PWM_A: now also U4.2 (PWMA)
- net PWM_B: now also U4.16 (PWMB)
- net STBY/RESET: now also U4.14 (STBY/RESET)
- new net: C9.1, R11.2, U4.11 (REF)
- new net: C8.1, RRCOFF.1
- new net: ROFF.2, RRCOFF.2, U4.12 (TOFF)
- new net: RsnsA.2, U4.4 (SENSEA)
- new net: R10.1, U4.9 (SENSEB)
- new net: C7.1, REN.2, U4.13 (EN/FLT)
- new net +3.3V: R11.1
- new net +BATT: C_Pol.1, Cs.1, U4.6 (VS)
- new net GND: C7.2, C8.2, C9.2, C_Pol.2, Cs.2, R10.2, ROFF.1, RsnsA.1, U4.7 (GND)

Commit message: test
Parts:
- removed C_Pol: 20µ, symbol Device:C_Polarized
- removed Cs: 2.2µ, symbol Device:C
- added C15: 2.2µF, Capacitor_SMD:C_0603_1608Metric, symbol Device:C
- C7, C8, C9: footprint (none) -> Capacitor_SMD:C_0603_1608Metric
- R10, R11: footprint (none) -> Resistor_SMD:R_0603_1608Metric
- R25: renamed from REN; footprint (none) -> Resistor_SMD:R_0603_1608Metric
- ROFF1: renamed from ROFF; footprint (none) -> Resistor_SMD:R_0603_1608Metric
- RRCOFF2: renamed from RRCOFF; footprint (none) -> Resistor_SMD:R_0603_1608Metric
- RsnsA1: renamed from RsnsA; footprint (none) -> Resistor_SMD:R_0603_1608Metric
Connections:
- net +BATT: now also C15.1
- net GND: now also U4.17 (EPAD), C15.2
- net FAULT: now reaches C7.1, R25.2, U4.13 (EN/FLT)
Other:
- moved on the sheet: RsnsA1
