File: minimouse.kicad_pcb (KiCad board)
At the start: 2 copper layers, 90 x 85 mm, 22 parts, among them J1 Conn_ARM_JTAG_SWD_10, J5 Conn_01x02, M1 N20_encoder, M2 N20_encoder, U1 STM32F030C8Tx, U4 HC-SR04

Commit message: test
Parts:
- added C10: 2.2µF, Capacitor_SMD:C_0603_1608Metric, F.Cu at (154.8, 119.7)
- added C11: 2.2µF, Capacitor_SMD:C_0603_1608Metric, F.Cu at (150.2, 117.7)
- added C12: 2.2µF, Capacitor_SMD:C_0603_1608Metric, F.Cu at (186.6, 90.5)
- added C15: 2.2µF, Capacitor_SMD:C_0603_1608Metric, F.Cu at (204.7, 64.3)
- added C16: 2.2µF, Capacitor_SMD:C_0603_1608Metric, F.Cu at (123.4, 82.1)
- added C17: 2.2µF, Capacitor_SMD:C_0603_1608Metric, F.Cu at (176.2, 89.5)
- added C18: 2.2µF, Capacitor_SMD:C_0603_1608Metric, F.Cu at (146.4, 56.9)
- added C7: 10n, Capacitor_SMD:C_0603_1608Metric, F.Cu at (204.7, 56.7)
- added C8: 22n, Capacitor_SMD:C_0603_1608Metric, F.Cu at (204.7, 59.2)
- added C9: C, Capacitor_SMD:C_0603_1608Metric, F.Cu at (204.7, 61.8)
- added D1: LED, LED_SMD:LED_0603_1608Metric, F.Cu at (145.8, 122.4)
- added J2: Conn_01x04, Connector_PinHeader_2.54mm:PinHeader_1x04_P2.54mm_Vertical, F.Cu at (180.0, 89.1)
- added J3: Conn_01x06, Connector_PinHeader_2.54mm:PinHeader_1x06_P2.54mm_Vertical, F.Cu at (169.8, 98.8)
- added J4: Conn_01x06, Connector_PinHeader_2.54mm:PinHeader_1x06_P2.54mm_Vertical, F.Cu at (139.8, 88.5)
- added R10: 330m, Resistor_SMD:R_0603_1608Metric, F.Cu at (203.8, 70.7)
- added R11: 10k, Resistor_SMD:R_0603_1608Metric, F.Cu at (208.7, 56.7)
- added R12: 100, Resistor_SMD:R_0603_1608Metric, F.Cu at (176.2, 93.3)
- added R13: 100, Resistor_SMD:R_0603_1608Metric, F.Cu at (170.6, 61.7)
- added R14: 100, Resistor_SMD:R_0603_1608Metric, F.Cu at (144.6, 118.2)
- added R15: 100, Resistor_SMD:R_0603_1608Metric, F.Cu at (165.0, 93.3)
- added R16: 100, Resistor_SMD:R_0603_1608Metric, F.Cu at (145.6, 81.9)
- added R17: 100, Resistor_SMD:R_0603_1608Metric, F.Cu at (165.0, 96.7)
- added R18: 100, Resistor_SMD:R_0603_1608Metric, F.Cu at (145.6, 80.3)
- added R19: 100, Resistor_SMD:R_0603_1608Metric, F.Cu at (152.0, 70.7)
- added R25: 18k, Resistor_SMD:R_0603_1608Metric, F.Cu at (208.7, 59.2)
- added ROFF1: 47k, Resistor_SMD:R_0603_1608Metric, F.Cu at (208.7, 61.8)
- added RRCOFF2: 1k, Resistor_SMD:R_0603_1608Metric, F.Cu at (208.7, 64.3)
- added RsnsA1: 330m, Resistor_SMD:R_0603_1608Metric, F.Cu at (207.8, 70.7)
- added U2: HC-SR04, minimouse:HC-SR04, F.Cu at (156.0, 57.2)
- added U3: LP5907MFX-3.3, Package_TO_SOT_SMD:SOT-23-5, F.Cu at (150.2, 121.7)
- U4: value HC-SR04 -> STSPIN240; footprint minimouse:HC-SR04 -> Package_DFN_QFN:VQFN-16-1EP_3x3mm_P0.5mm_EP1.8x1.8mm
- moved C1 68.8 mm to (199.2, 52.3), turned to -90 degrees
- moved U4 28.8 mm to (153.8, 97.7), turned to 180 degrees
- moved C5 23.0 mm to (137.2, 70.7), turned to 0 degrees
- moved C4 19.0 mm to (163.2, 77.0)
- moved R1 15.7 mm to (162.4, 72.1), turned to 180 degrees
- moved R5 15.7 mm to (151.4, 84.7)
- moved R4 15.7 mm to (149.8, 84.7)
- moved R3 15.6 mm to (148.2, 84.7), turned to 90 degrees
- moved R7 15.0 mm to (154.6, 84.7), turned to -90 degrees
- moved R6 14.9 mm to (153.0, 84.7), turned to -90 degrees
- moved C3 14.9 mm to (143.2, 71.9), turned to -90 degrees
- moved C2 14.7 mm to (144.9, 68.1)
- moved C6 14.7 mm to (143.3, 68.1)
- moved R8 12.9 mm to (156.2, 69.1)
- moved U1 12.2 mm to (152.6, 77.7)
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Connections:
- U1 pad 43: /mcu/UART1_RX -> /external_uart/EXT_UART_TX
- U4 pad 1: GND -> /mcu/OUT_A4
- U4 pad 2: /mcu/OUT_B9 -> /mcu/TIM15_CH1
- U4 pad 3: Net-(U4-ECHO) -> /motorB/MA
- U4 pad 4: +3V3 -> Net-(U4-SENSEA)

Commit message: just save
Parts:
- moved R11 70.9 mm to (147.4, 92.3), turned to -90 degrees
- moved C1 63.6 mm to (138.8, 72.3), turned to 90 degrees
- moved C9 63.3 mm to (152.5, 97.6), turned to -90 degrees
- moved RRCOFF2 60.3 mm to (158.4, 97.5), turned to 90 degrees
- moved ROFF1 60.3 mm to (160.2, 97.5), turned to 90 degrees
- moved C7 57.7 mm to (164.8, 98.5), turned to 90 degrees
- moved C8 57.3 mm to (162.2, 97.7), turned to 90 degrees
- moved R25 55.4 mm to (160.0, 85.7), turned to -90 degrees
- moved R10 55.2 mm to (155.3, 97.1), turned to 180 degrees
- moved C15 53.9 mm to (157.4, 90.1), turned to 180 degrees
- moved RsnsA1 49.8 mm to (162.9, 92.1), turned to 90 degrees
- moved R14 42.8 mm to (184.0, 101.5), turned to -90 degrees
- moved D1 38.5 mm to (179.2, 103.3), turned to 0 degrees
- moved C10 37.2 mm to (185.0, 97.9)
- moved C11 37.2 mm to (179.8, 95.2)
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Routing:
- net GND: track 0.00 -> 345.2 mm
- net +BATT: track 0.00 -> 111.8 mm
- net +3.3V: track 0.00 -> 40.0 mm
- net /external_uart/EXT_UART_TX: track 0.00 -> 34.7 mm
- net /mcu/TIM3_CH1: track 0.00 -> 31.7 mm
- net /mcu/IN_B2: track 0.00 -> 30.9 mm
- net /motorA/MA: track 0.00 -> 24.4 mm
- net Net-(U2-ECHO): track 0.00 -> 22.5 mm
- net /mcu/OUT_B9: track 0.00 -> 22.1 mm
- net /mcu/BOOT0: track 0.00 -> 18.6 mm
- net Net-(J4-Pin_3): track 0.00 -> 15.5 mm
- net /mcu/TIM2_CH1: track 0.00 -> 10.8 mm
- net Net-(J4-Pin_4): track 0.00 -> 9.88 mm
- net Net-(J2-Pin_3): track 0.00 -> 7.87 mm
- net Net-(C8-Pad1): track 0.00 -> 6.73 mm
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
Commit message: heyo
Parts:
- removed R13: 100, Resistor_SMD:R_0603_1608Metric
- moved C18 40.4 mm to (164.8, 57.4)
- moved RsnsA1 27.1 mm to (135.9, 95.0)
- moved C7 21.2 mm to (148.2, 85.3)
- moved C1 18.0 mm to (156.8, 70.5)
- moved C2 17.9 mm to (149.0, 83.1), turned to 0 degrees
- moved C15 16.3 mm to (142.4, 96.6), turned to 0 degrees
- moved U4 15.8 mm to (142.3, 92.9), turned to 0 degrees
- moved ROFF1 13.4 mm to (151.9, 87.0), turned to 180 degrees
- moved C8 12.9 mm to (151.8, 90.1), turned to 180 degrees
- moved RRCOFF2 11.1 mm to (151.8, 88.6), turned to 180 degrees
- moved R11 8.70 mm to (156.1, 92.1)
- moved U2 8.41 mm to (150.0, 56.7)
- moved C16 8.19 mm to (127.5, 74.3), turned to 90 degrees
- moved C4 7.39 mm to (139.4, 71.8), turned to 90 degrees
- moved R10 7.18 mm to (148.4, 95.4), turned to -90 degrees
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Connections:
- R8 pad 1: /mcu/UART1_TX -> /external_uart/EXT_UART_RX
- U2 pad 4: +3.3V -> +BATT
Routing:
- net GND: track 345.2 -> 28.7 mm, vias 0 -> 18
- net +BATT: track 111.8 -> 234.1 mm
- net /motorA/MB: track 0.00 -> 55.2 mm
- net +3.3V: track 40.0 -> 93.0 mm
- net /external_uart/EXT_UART_RX: track 0.00 -> 49.5 mm
- net /motorB/MB: track 0.00 -> 47.0 mm
- net /mcu/TIM3_CH2: track 0.77 -> 30.7 mm, vias 0 -> 2
- net /mcu/SWDIO: track 0.00 -> 28.1 mm
- net /motorB/MA: track 0.14 -> 20.2 mm
- net /mcu/OUT_B1: track 0.00 -> 14.3 mm
- net Net-(U4-REF): track 0.00 -> 12.4 mm
- net Net-(J3-Pin_4): track 0.00 -> 10.8 mm
- net Net-(U4-TOFF): track 0.00 -> 10.5 mm
- net /motorA/MA: track 24.4 -> 34.8 mm
- net /mcu/SWO: track 0.00 -> 10.2 mm
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- added copper zone on B.Cu, net GND
